File: Mcu - data logger.kicad_pcb (KiCad board)
At the start: 2 copper layers, 0 parts

Commit message: Update MCU data logger PCB and project
Parts:
- added BT1: Battery, Package_TO_SOT_SMD:SOT-23-5, F.Cu at (41.1, 52.0)
- added C1: 0.1uF, Capacitor_SMD:C_0805_2012Metric, F.Cu at (60.0, 39.0)
- added C2: 22 pf, Capacitor_SMD:C_0805_2012Metric, F.Cu at (78.5, 59.0)
- added C3: 22 pf, Capacitor_SMD:C_0805_2012Metric, F.Cu at (65.0, 39.0)
- added C4: C, Capacitor_SMD:C_0805_2012Metric, F.Cu at (78.5, 64.5)
- added C5: 100 nF, Capacitor_SMD:C_0805_2012Metric, F.Cu at (70.0, 39.0)
- added D1: LED, LED_SMD:LED_0805_2012Metric, F.Cu at (83.4, 39.0)
- added D2: LED, LED_SMD:LED_0805_2012Metric, F.Cu at (78.5, 39.0)
- added H1: MountingHole, MountingHole:MountingHole_2.1mm, F.Cu at (40.5, 39.5)
- added H2: MountingHole, MountingHole:MountingHole_2.1mm, F.Cu at (40.5, 75.5)
- added H3: MountingHole, MountingHole:MountingHole_2.1mm, F.Cu at (91.0, 39.5)
- added H4: MountingHole, MountingHole:MountingHole_2.1mm, F.Cu at (91.0, 75.5)
- added J1: Conn_01x04_Pin, Connector_PinHeader_2.54mm:PinHeader_1x04_P2.54mm_Vertical, F.Cu at (91.5, 60.5)
- added J2: Conn_01x04_Pin, Connector_PinHeader_2.54mm:PinHeader_1x04_P2.54mm_Vertical, F.Cu at (73.5, 76.0)
- added J3: Conn_01x09_Pin, Connector_PinHeader_2.54mm:PinHeader_1x09_P2.54mm_Vertical, F.Cu at (45.5, 76.0)
- added J4: Conn_02x03_Odd_Even, Connector_PinHeader_2.54mm:PinHeader_2x03_P2.54mm_Vertical, F.Cu at (89.0, 48.5)
- added R1: 10 K, Resistor_SMD:R_0805_2012Metric, F.Cu at (48.4, 72.0)
- added R2: 10 K, Resistor_SMD:R_0805_2012Metric, F.Cu at (54.0, 72.0)
- added R3: 4.7K, Resistor_SMD:R_0805_2012Metric, F.Cu at (78.5, 54.0)
- added R4: 4.7K, Resistor_SMD:R_0805_2012Metric, F.Cu at (78.4, 49.0)
- added R5: 330, Resistor_SMD:R_0805_2012Metric, F.Cu at (78.4, 44.0)
- added R6: 10 K, Resistor_SMD:R_0805_2012Metric, F.Cu at (83.4, 49.0)
- added R7: 330, Resistor_SMD:R_0805_2012Metric, F.Cu at (83.4, 44.0)
- added U1: 24LC1025, Package_SO:SOIC-8_5.3x6.2mm_P1.27mm, F.Cu at (52.0, 45.0)
- added U2: 24LC1025, Package_SO:SOIC-8_3.9x4.9mm_P1.27mm, F.Cu at (52.0, 55.5)
- added U3: DS1337, Footprints:DIL08-ROUND, F.Cu at (52.5, 65.0)
- added U5: ATMEGA328P-AU, Footprints:QFP80P900X900X120-32N, F.Cu at (65.0, 52.5)
- added Y1: 32.768 KHz, Crystal:Crystal_SMD_5032-2Pin_5.0x3.2mm_HandSoldering, F.Cu at (41.5, 62.1)
- added Y2: 16 MHz, Crystal:Crystal_SMD_5032-2Pin_5.0x3.2mm_HandSoldering, F.Cu at (65.0, 66.0)
Other:
- board outline added: 59.4 x 41 mm

Commit message: Routes
Parts:
- moved U2 14.5 mm to (51.0, 41.0)
- moved U1 7.02 mm to (51.5, 52.0)
- moved C2 6.00 mm to (78.5, 65.0), turned to 180 degrees
- moved D2 5.06 mm to (83.6, 39.0)
- moved C4 5.00 mm to (78.5, 59.5), turned to 180 degrees
- moved D1 4.94 mm to (78.5, 39.0)
- turned R2 to 180 degrees
- turned R3 to 180 degrees
- turned R4 to 180 degrees
- turned R5 to 180 degrees
- turned U3 to -90 degrees
- turned Y1 to 90 degrees
- turned Y2 to 180 degrees
Routing:
- net /SCK: track 0.00 -> 159.9 mm, vias 0 -> 5
- net /Vcc: track 0.00 -> 131.3 mm, vias 0 -> 4
- net /SDA: track 0.00 -> 89.3 mm, vias 0 -> 2
- net Net-(BT1-+): track 0.00 -> 71.4 mm, vias 0 -> 5
- net GND: track 0.00 -> 68.2 mm, vias 0 -> 6
- net /TX: track 0.00 -> 36.5 mm, vias 0 -> 1
- net /D2: track 0.00 -> 36.4 mm, vias 0 -> 1
- net /MISO: track 0.00 -> 35.8 mm, vias 0 -> 1
- net /D3: track 0.00 -> 35.7 mm
- net Net-(U5-PB7): track 0.00 -> 35.6 mm, vias 0 -> 4
- net /RX: track 0.00 -> 33.8 mm, vias 0 -> 1
- net /D4: track 0.00 -> 33.2 mm
- net /MOSI: track 0.00 -> 30.1 mm
- net /RESET: track 0.00 -> 30.0 mm, vias 0 -> 4
- net /D5: track 0.00 -> 22.0 mm, vias 0 -> 1
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