File: Mcu - data logger.kicad_pcb (KiCad board)
At the start: 2 copper layers, 52.8 x 34.3 mm, 29 parts, among them J1 Conn_01x04_Pin, J2 Conn_01x09_Pin, J3 Conn_01x04_Pin, J4 Conn_02x03_Odd_Even, U1 24LC1025, U2 DS1337S_, U3 24LC1025, U4 ATMEGA328P-AU, Y1 32.768 KHz, Y2 16 MHz

Commit message: Some more fixes
Other:
- board text added: "2"
- board text added: "3"
- board text added: "4"
- board text added: "5"
- board text added: "6"
- board text added: "7"
- board text added: "8"
- board text added: "GND"
- board text added: "GPIO"
- board text added: "I2C"
- board text added: "ICSP"
- board text added: "RX"
- board text added: "SCK"
- board text added: "SDA"
- board text added: "Serial"
- board text added: "TX"
- board text added: "VCC"
