File: Mcu - data logger.kicad_sch (KiCad schematic)
At the start: 25 parts, among them U1 24LC1025, U2 24LC1025, U3 DS1337, U5 ATMEGA328P-AU, Y1 32.768 KHz, Y2 16 MHz

Commit message: schmatic design done
Other:
- note added: "EEPROM"
- note added: "MCU"
- note added: "Mouting"
- note added: "Real time clock"
- moved on the sheet: H1, H2, H3, H4, R3, R4, U1, U2

Commit message: Routes
Parts:
- R5: value 300 -> 330
Changed lines of the file:
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@@
 			)
 		)
-		(property "Value" "300"
+		(property "Value" "330"
 			(at 153.67 35.56 90)
 			(show_name no)
