File: _restore_backup_2026-09-23T10-11-36-198/Mcu - data logger.kicad_sch (KiCad schematic)
At the start: 25 parts, among them U1 24LC1025, U2 24LC1025, U3 DS1337, U5 ATMEGA328P-AU, Y1 32.768 KHz, Y2 16 MHz

Commit message: schematic work
Parts:
- removed U5: ATMEGA328P-AU, Footprints:QFP80P900X900X120-32N, symbol ATMEGA328P-AU:ATMEGA328P-AU
- added U4: ATMEGA328P-AU, Footprints:QFP80P900X900X120-32N, symbol ATMEGA328-AU:ATMEGA328P-AU
Connections:
- net D2: now also U4.32 (PD2)
- net D3: now also U4.1 (PD3)
- net D4: now also U4.2 (PD4)
- net D5: now also U4.9 (PD5)
- net D6: now also U4.10 (PD6)
- net D7: now also U4.11 (PD7)
- net D8: now also U4.12 (PB0)
- net GND: now also U4.21 (GND), U4.3 (GND), U4.5 (GND)
- net MISO: now also U4.16 (PB4)
- net MOSI: now also U4.15 (PB3)
- net RESET: now also U4.29 (PC6/~{RESET})
- net RX: now also U4.31 (PD1)
- net SCK: now also U4.17 (PB5), U4.28 (PC5)
- net SDA: now also U4.27 (PC4)
- net TX: now also U4.30 (PD0)
- net at C4.2: now also U4.20 (AREF)
- net at BT1.1 (+), C5.1, D2.2 (A): now also U4.18 (AVCC), U4.4 (VCC)
- net at C2.2, Y2.2: now also U4.7 (PB6)
- net at C3.2, Y2.1: now also U4.8 (PB7)
